File: GaN_pwr_delivery_module.kicad_sch (KiCad schematic)
At the start: 41 parts, among them J1 Conn_01x02_Pin, J2 gateBias, Q1 AONS66920, Q2 2N7002, U1 LT4256-1CS8, U2 TPS7A1650DGNR, U32 LM2662MX_NOPB

Commit message: init ideas
Parts:
- removed Q2: 2N7002, Package_TO_SOT_SMD:SOT-23, symbol Transistor_FET:2N7002
- removed R3, R4: 100k, symbol Device:R
- removed R5: 27k, symbol Device:R
- added C44: 10nF, Capacitor_SMD:C_0805_2012Metric_Pad1.18x1.45mm_HandSolder, symbol Device:C
- added D34, D35: BAT54S, Package_TO_SOT_SMD:SOT-23, symbol Diode:BAT54S
- added J3: gateBias, Connector_Wire:SolderWire-0.1sqmm_1x02_P3.6mm_D0.4mm_OD1mm, symbol Connector:Conn_01x02_Pin
- added R35, R36: 10k, symbol Device:R
- added R39: 27k, symbol Device:R
- added R40: 1k, symbol Device:R
- added R41, R42, R43: R, symbol Device:R
- added U34: LM324, LM324DRG3:SOIC127P600X175-14N, symbol Amplifier_Operational:LM324
- C1: footprint (none) -> Capacitor_SMD:CP_Elec_3x5.3
- C2, C3, C4: footprint (none) -> Capacitor_SMD:C_0805_2012Metric
- R1: footprint (none) -> Resistor_SMD:R_0805_2012Metric
Connections:
- net +28V: now also J3.2 (Pin_2), R39.1, U34.4 (V+)
- net GND: now also C44.1, J3.1 (Pin_1), R40.2, R42.2, R43.2, U34.11 (V-), U34.3 (+)
- net isGateOn: now also U1.1 (UV), R41.2, R42.1
- net negGateV: now also R35.1
- new net: C44.2, D35.1 (A), R39.2, R40.1, U34.10 (+), U34.5 (+)
- new net: R35.2, R36.1, U34.2 (-)
- new net: D34.1 (A), R36.2, U34.1
- new net: R41.1, U34.8
- new net: D34.2 (K), R43.1, U34.6 (-)
- new net: D35.3 (COM), U34.7, U34.9 (-)
- no-connect marks 1 -> 3
Other:
- note added: "1V"
- note added: "R1 = R2 (V_out/V_ref_1.2 -1)"
- note removed: "R1 = R2 (V_out/V_ref -1)"
- note removed: "need to redesign"
- moved on the sheet: C1, C2, C3, C4, C5, D1, J1, Q1, R1, R2, R6, R7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
