File: GaN_pwr_delivery_module.kicad_sch (KiCad schematic)
At the start: 49 parts, among them J1 Conn_01x02_Pin, J2 gateBias, J3 gateBias, Q1 AONS66920, U1 LT4256-1CS8, U2 TPS7A1650DGNR, U32 LM2662MX_NOPB, U34 LM324

Commit message: init
Parts:
- removed R43: R, symbol Device:R
- added C42: C, symbol Device:C
- added D36: BAT54S, Package_TO_SOT_SMD:SOT-23, symbol Diode:BAT54S
- added R32: 100k, symbol Device:R
- added TP7: TestPoint, TestPoint:TestPoint_Pad_D1.5mm, symbol Connector:TestPoint
- R2: footprint Resistor_SMD:R_0603_1608Metric -> Resistor_SMD:R_0805_2012Metric
- R40: value 1k -> 500
- R6, R7: footprint (none) -> Resistor_SMD:R_0805_2012Metric
Connections:
- net +28V: now also R2.1; no longer Q1.5_8
- net GND: now also C42.2, D36.2 (K)
- net isGateOn: now also TP7.1
- net at D1.1 (K), Q1.4: now also U1.6 (GATE); no longer R2.2, U1.7 (SENSE)
- net at R36.2, U34.1: now also R32.1; no longer D34.1 (A)
- net at U34.6 (-): now also D34.1 (A), C42.1, R32.2; no longer D34.2 (K)
- new net: Q1.5_8, R2.2, U1.7 (SENSE)
- new net: D34.2 (K), D36.1 (A)
- no-connect marks 3 -> 4
Other:
- moved on the sheet: D34, R2

Commit message: init ideas
Parts:
- removed C38: 10nF, Capacitor_SMD:C_0805_2012Metric, symbol Device:C
- removed C39, C44: 10nF, Capacitor_SMD:C_0805_2012Metric_Pad1.18x1.45mm_HandSolder, symbol Device:C
- removed C40: 100uF, Capacitor_SMD:CP_Elec_3x5.3, symbol Device:C_Polarized
- removed C41: 1nF, Capacitor_SMD:C_0805_2012Metric, symbol Device:C
- removed C42: C, symbol Device:C
- removed D34, D35, D36: BAT54S, Package_TO_SOT_SMD:SOT-23, symbol Diode:BAT54S
- removed R10: 100k, Resistor_SMD:R_0805_2012Metric, symbol Device:R
- removed R32, R8: 100k, symbol Device:R
- removed R35, R36: 10k, symbol Device:R
- removed R39: 27k, symbol Device:R
- removed R40: 500, symbol Device:R
- removed R41, R42: R, symbol Device:R
- removed TP4, TP5: ~, TestPoint:TestPoint_Pad_D1.5mm, symbol Connector:TestPoint
- removed U2: TPS7A1650DGNR, TPS7A1650DGNR:SOP65P490X110-9N, symbol TPS7A1650DGNR:TPS7A1650DGNR
- removed U34: LM324, LM324DRG3:SOIC127P600X175-14N, symbol Amplifier_Operational:LM324
- added C1: 10nF, Capacitor_SMD:C_0805_2012Metric_Pad1.18x1.45mm_HandSolder, symbol Device:C
- added C11: 10nF, Capacitor_SMD:C_0805_2012Metric, symbol Device:C
- added C3: 100uF, Capacitor_SMD:CP_Elec_3x5.3, symbol Device:C_Polarized
- added D32: BAT54SW, Package_TO_SOT_SMD:SOT-323_SC-70, symbol Diode:BAT54SW
- added R2, R5: 100k, Resistor_SMD:R_0805_2012Metric, symbol Device:R
- added R3: 62k, Resistor_SMD:R_0805_2012Metric, symbol Device:R
- added R4: 10k, Resistor_SMD:R_0805_2012Metric, symbol Device:R
- added U1: LDO40LPURY, LDO40LPURY:SON95P300X300X100-7N, symbol LDO40LPURY:LDO40LPURY
- added U4: LM324, LM324DRG3:SOIC127P600X175-14N, symbol Amplifier_Operational:LM324
- J1: renamed from J3; value gateBias -> dcConn
- J2: value gateBias -> gateConn
- J3: renamed from J1; value Conn_01x02_Pin -> drainConn
- JP1: renamed from JP32; value SolderJumper_2_Open -> OSC_switch
- R9: value 30k -> 100k
- RV1: value 100k -> 200k
- renumbered C33 to C10, C37 to C12, C35 to C13, C5 to C14, C1 to C2, C2 to C4, C36 to C5, C3 to C6, C34 to C7, C4 to C8, C32 to C9, R7 to R6, R6 to R7, R2 to R8, TP6 to TP3, TP7 to TP4, TP3 to TP5, U32 to U2, U1 to U3
Connections:
- net +28V: now also C1.1, C3.1, U1.2 (EN), U1.3 (VIN), U4.4 (V+)
- net GND: now also C1.2, C3.2, D32.2 (K), U1.1 (GND), U4.11 (V-)
- net isGateOn: now also R9.1, R5.1, U4.1
- net negGateV: now also R4.2
- net posGateV: now also C11.1, R2.1, U1.4 (VOUT), U1.5 (VSENSE)
- net at RV1.1: now also R3.2; no longer R9.2
- new net: C11.2, R2.2, R3.1, U1.6 (ADJ)
- new net: D32.1 (A), R9.2, U4.3 (+)
- new net: R4.1, R5.2, U4.2 (-)
- no-connect marks 4 -> 11
Other:
- note added: "Vout = V_ref_1.2*(1+R2/R1)"
- note removed: "1V"
- note removed: "R1 = R2 (V_out/V_ref_1.2 -1)"
- moved on the sheet: C10, C12, C13, C14, C2, C4, C5, C6, C7, C8, C9, D1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

Commit message: init idea
Parts:
- removed U1: LDO40LPURY, LDO40LPURY:SON95P300X300X100-7N, symbol LDO40LPURY:LDO40LPURY
- added U1: LDO40LPURY, Package_DFN_QFN:DFN-6-1EP_3x3mm_P0.95mm_EP1.7x2.6mm, symbol Regulator_Linear:LDO40LPURY
- C13, C3: now not fitted; now left out of the parts list
Connections:
- net +28V: now also U1.2 (EN), U1.3 (Vin)
- net GND: now also U1.1 (GND), U1.7 (GND)
- net posGateV: now also U1.4 (Vout), U1.5 (Vsense)
- net at C11.2, R2.2, R3.1: now also U1.6 (ADJ)
Other:
- moved on the sheet: C11, R2, R3, RV1, TP3

Commit message: init
Parts:
- TP3: value ~ -> TestPoint
Changed lines of the file:
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@@
 			)
 		)
-		(property "Value" "~"
-			(at 99.06 67.8181 0)
+		(property "Value" "TestPoint"
+			(at 96.012 67.818 0)
 			(effects
 				(font

Commit message: init ideas
Connections:
- net at U4.5 (+): now also U4.6 (-)
Other:
- moved on the sheet: C1, C10, C11, C12, C13, C14, C2, C3, C4, C5, C6, C7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

Commit message: POC
Parts:
- added R10: 100k, Resistor_SMD:R_0805_2012Metric, symbol Device:R
- added TP6: TestPoint, TestPoint:TestPoint_Pad_D1.5mm, symbol Connector:TestPoint
- C13, C3: value 100uF -> 10uF; footprint Capacitor_SMD:CP_Elec_3x5.3 -> Capacitor_SMD:CP_Elec_6.3x9.9
- C2: footprint Capacitor_SMD:CP_Elec_3x5.3 -> Capacitor_SMD:CP_Elec_6.3x9.9
- C7: value 100uF -> 10uF; footprint Capacitor_SMD:CP_Elec_3x5.3 -> Capacitor_SMD:CP_Elec_6.3x9.9; now not fitted; now left out of the parts list
Connections:
- net GND: now also R10.2
- net isGateOn: now also R10.1
- net negGateV: now also TP6.1
