File: GaN_pwr_delivery_module.kicad_pcb (KiCad board)
At the start: 2 copper layers, 19 parts, among them J2 gateBias, U2 TPS7A1650DGNR, U32 LM2662MX_NOPB

Commit message: init ideas
Parts:
- added C1: 100uF, Capacitor_SMD:CP_Elec_3x5.3, F.Cu at (230.9, 125.3)
- added C2: 100nF, Capacitor_SMD:C_0805_2012Metric, F.Cu at (230.9, 128.6)
- added C3: 10nF, Capacitor_SMD:C_0805_2012Metric, F.Cu at (230.9, 130.9)
- added C4: 1nF, Capacitor_SMD:C_0805_2012Metric, F.Cu at (230.9, 133.2)
- added J3: gateBias, Connector_Wire:SolderWire-0.1sqmm_1x02_P3.6mm_D0.4mm_OD1mm, F.Cu at (229.1, 135.8)
- added R1: 100k, Resistor_SMD:R_0805_2012Metric, F.Cu at (230.9, 121.8)
- moved RV1 10.2 mm to (248.7, 113.3)
- moved C39 8.98 mm to (245.5, 121.0), turned to 0 degrees
- moved C40 8.92 mm to (245.5, 124.0), turned to 0 degrees
- moved TP4 7.07 mm to (241.0, 122.9)
- moved TP5 6.27 mm to (252.6, 120.0)
- moved R9 1.89 mm to (252.4, 116.7), turned to 90 degrees
- moved C32 1.40 mm to (240.4, 129.9)
- moved C33 1.40 mm to (237.7, 129.9)
Routing:
- net +28V: track 13.3 -> 35.1 mm
- net GND: track 18.6 -> 3.28 mm, vias 26 -> 257
- net Net-(R9-Pad2): track 0.00 -> 6.04 mm
- net Net-(JP32-B): track 12.4 -> 8.01 mm
- net Net-(U2-FB/DNC): track 6.24 -> 8.67 mm
- net Net-(U2-PG): track 11.1 -> 10.5 mm
- net (no net): vias 16 -> 17

Commit message: init pcb
Routing:
- net GND: track 3.28 -> 8.39 mm, vias 257 -> 265
- net (no net): vias 17 -> 16
Changed lines of the file:
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@@
 			(psa4output no)
 			(plot_black_and_white yes)
-			(plotinvisibletext no)
 			(sketchpadsonfab no)
 			(plotpadnumbers no)
@@
 	)
 	(via
-		(at 242.525 129.9)
-		(size 0.2)
-		(drill 0.1)
-		(layers "F.Cu" "B.Cu")
-		(free yes)
-		(net 0)
-	)
-	(via
 		(at 244.063333 117.3)
 		(size 0.2)
@@
 	)
 	(segment
+		(start 248.925 129.935)
+		(end 250.350283 129.935)
+		(width 0.3)
+		(layer "F.Cu")
+		(net 1)
+	)
+	(segment
 		(start 246.6 122.3875)
 		(end 247.025 122.8125)
@@
 	)
 	(segment
+		(start 246.4 117.05)
+		(end 246.4 115.7)
+		(width 0.2)
+		(layer "F.Cu")
+		(net 1)
+	)
+	(segment
 		(start 246.6 121.0125)
 		(end 246.6 122.3875)
@@
 		(net 1)
 	)
+	(segment
+		(start 243.985 129.935)
+		(end 241.65 129.935)
+		(width 0.3)
+		(layer "F.Cu")
+		(net 1)
+	)
 	(via
 		(at 234.35 136.25)
@@
 	)
 	(via
-		(at 238.7 129.9)
+		(at 238.675 129.935)
 		(size 0.2)
 		(drill 0.1)
@@
 	)
 	(via
-		(at 250.35 129.908333)
+		(at 250.350283 129.935)
 		(size 0.2)
 		(drill 0.1)
@@
 	)
 	(via
-		(at 250.7 129.5)
+		(at 250.700283 129.526667)
 		(size 0.2)
 		(drill 0.1)
@@
 	)
 	(via
-		(at 250.95 129.908333)
+		(at 250.950283 129.935)
 		(size 0.2)
 		(drill 0.1)
@@
 	)
 	(via
-		(at 239.55 129.9)
+		(at 239.525 129.935)
 		(size 0.2)
 		(drill 0.1)
@@
 	)
 	(via
-		(at 251.3 129.5)
+		(at 246.094181 115.3)
+		(size 0.2)
+		(drill 0.1)
+		(layers "F.Cu" "B.Cu")
+		(net 1)
+	)
+	(via
+		(at 251.300283 129.526667)
 		(size 0.2)
 		(drill 0.1)
@@
 	)
 	(via
-		(at 242.1 129.9)
+		(at 242.075 129.935)
 		(size 0.2)
 		(drill 0.1)
@@
 	)
 	(via
-		(at 241.25 129.9)
+		(at 241.225 129.935)
 		(size 0.2)
 		(drill 0.1)
@@
 	)
 	(via
-		(at 238.325 129.9)
+		(at 238.3 129.935)
 		(size 0.2)
 		(drill 0.1)
@@
 	)
 	(via
+		(at 246.7 116.2)
+		(size 0.2)
+		(drill 0.1)
+		(layers "F.Cu" "B.Cu")
+		(net 1)
+	)
+	(via
 		(at 237.625 132.1)
 		(size 0.2)
@@
 	)
 	(via
+		(at 242.5 129.935)
+		(size 0.2)
+		(drill 0.1)
+		(layers "F.Cu" "B.Cu")
+		(free yes)
+		(net 1)
+	)
+	(via
 		(at 246.05 119.8)
 		(size 0.2)
@@
 	)
 	(via
-		(at 237.9 129.9)
+		(at 237.875 129.935)
 		(size 0.2)
 		(drill 0.1)
@@
 	)
 	(via
+		(at 246.1 116.2)
+		(size 0.2)
+		(drill 0.1)
+		(layers "F.Cu" "B.Cu")
+		(net 1)
+	)
+	(via
 		(at 227.5 135.825)
 		(size 0.2)
@@
 	)
 	(via
-		(at 240.825 129.9)
+		(at 240.8 129.935)
 		(size 0.2)
 		(drill 0.1)
@@
 	)
 	(via
+		(at 247 115.7)
+		(size 0.2)
+		(drill 0.1)
+		(layers "F.Cu" "B.Cu")
+		(net 1)
+	)
+	(via
 		(at 236.771667 127.8)
 		(size 0.2)
@@
 	)
 	(via
+		(at 245.8 115.7)
+		(size 0.2)
+		(drill 0.1)
+		(layers "F.Cu" "B.Cu")
+		(net 1)
+	)
+	(via
 		(at 228.8 128.575)
 		(size 0.2)
@@
 	)
 	(via
-		(at 237.05 129.9)
+		(at 237.025 129.935)
 		(size 0.2)
 		(drill 0.1)
@@
 	)
 	(via
-		(at 251.3 130.3)
+		(at 251.300283 130.326667)
 		(size 0.2)
 		(drill 0.1)
@@
 	)
 	(via
+		(at 246.4 115.7)
+		(size 0.2)
+		(drill 0.1)
+		(layers "F.Cu" "B.Cu")
+		(net 1)
+	)
+	(via
 		(at 238.475 132.1)
 		(size 0.2)
@@
 	)
 	(via
-		(at 241.675 129.9)
+		(at 241.65 129.935)
 		(size 0.2)
 		(drill 0.1)
@@
 	)
 	(via
-		(at 239.125 129.9)
+		(at 239.1 129.935)
 		(size 0.2)
 		(drill 0.1)
@@
 	)
 	(via
-		(at 240.4 129.9)
+		(at 240.375 129.935)
 		(size 0.2)
 		(drill 0.1)
@@
 	)
 	(via
-		(at 251.55 129.908333)
+		(at 251.550283 129.935)
 		(size 0.2)
 		(drill 0.1)
@@
 	)
 	(via
-		(at 250.7 130.3)
+		(at 250.700283 130.326667)
+		(size 0.2)
+		(drill 0.1)
+		(layers "F.Cu" "B.Cu")
+		(net 1)
+	)
+	(via
+		(at 246.694181 115.3)
 		(size 0.2)
 		(drill 0.1)
@@
 	)
 	(via
-		(at 239.975 129.9)
+		(at 239.95 129.935)
 		(size 0.2)
 		(drill 0.1)
@@
 	)
 	(via
-		(at 237.475 129.9)
+		(at 237.45 129.935)
 		(size 0.2)
 		(drill 0.1)

Commit message: init
Parts:
- added C5: 27nF, Capacitor_SMD:C_0805_2012Metric_Pad1.18x1.45mm_HandSolder, F.Cu at (227.5, 124.7)
- added D1: BZV55C30, Diode_SMD:D_MiniMELF, F.Cu at (232.1, 129.5)
- added J1: Conn_01x02_Pin, Connector_Wire:SolderWire-0.1sqmm_1x02_P3.6mm_D0.4mm_OD1mm, F.Cu at (240.1, 135.9)
- added Q1: AONS66920, AONS66920:TRANS_AONS66920, F.Cu at (226.6, 129.3)
- added R2: 0.027, Resistor_SMD:R_0805_2012Metric, F.Cu at (221.1, 127.0)
- added R6: 100k, Resistor_SMD:R_0805_2012Metric, F.Cu at (234.8, 130.3)
- added R7: 27k, Resistor_SMD:R_0805_2012Metric, F.Cu at (234.8, 124.7)
- added TP7: TestPoint, TestPoint:TestPoint_Pad_D1.5mm, F.Cu at (222.7, 118.0)
- added U1: LT4256-1CS8, LT4256-1CS8:SO-8_S, F.Cu at (227.3, 121.0)
- moved J3 24.2 mm to (224.8, 112.0), turned to -90 degrees
- moved C4 19.7 mm to (227.4, 113.8), turned to 90 degrees
- moved C3 17.1 mm to (229.7, 113.8), turned to 90 degrees
- moved C2 14.8 mm to (232.0, 113.8), turned to 90 degrees
- moved C1 12.3 mm to (235.3, 113.8), turned to 90 degrees
- moved R1 11.2 mm to (238.8, 113.8), turned to 90 degrees
- moved R9 2.56 mm to (252.9, 114.2)
Routing:
- net Net-(U1-SENSE): track 0.00 -> 23.1 mm, vias 0 -> 2
- net Net-(U1-FB): track 0.00 -> 21.9 mm, vias 0 -> 2
- net +28V: track 35.1 -> 56.3 mm
- net drainV: track 0.00 -> 18.6 mm
- net Net-(D1-K): track 0.00 -> 10.7 mm
- net Net-(U1-TIMER): track 0.00 -> 5.93 mm
- net Net-(U2-FB/DNC): track 8.67 -> 12.7 mm, vias 0 -> 2
- net Net-(R9-Pad2): track 6.04 -> 4.17 mm
- net isGateOn: track 0.00 -> 1.82 mm
- net GND: vias 265 -> 289
- net (no net): vias 16 -> 0
- added copper zone on B.Cu, net GND

Commit message: init ideas
Parts:
- removed C32, C33: 47uF, Capacitor_SMD:C_0805_2012Metric_Pad1.18x1.45mm_HandSolder
- removed C34, C35, C40: 100uF, Capacitor_SMD:CP_Elec_3x5.3
- removed C36, C37, C39: 10nF, Capacitor_SMD:C_0805_2012Metric_Pad1.18x1.45mm_HandSolder
- removed C38: 10nF, Capacitor_SMD:C_0805_2012Metric
- removed JP32: SolderJumper_2_Open, Jumper:SolderJumper-2_P1.3mm_Open_RoundedPad1.0x1.5mm
- removed R10: 100k, Resistor_SMD:R_0805_2012Metric
- removed TP4, TP5, TP6: ~, TestPoint:TestPoint_Pad_D1.5mm
- removed TP7: TestPoint, TestPoint:TestPoint_Pad_D1.5mm
- removed U32: LM2662MX_NOPB, LM2662MX_NOPB:SOIC127P599X175-8N
- added C10: 47uF, Capacitor_SMD:C_0805_2012Metric_Pad1.18x1.45mm_HandSolder, F.Cu at (130.4, 104.8)
- added C11: 10nF, Capacitor_SMD:C_0805_2012Metric, F.Cu at (139.5, 88.2)
- added C12: 10nF, Capacitor_SMD:C_0805_2012Metric_Pad1.18x1.45mm_HandSolder, F.Cu at (140.2, 108.8)
- added C13: 100uF, Capacitor_SMD:CP_Elec_3x5.3, F.Cu at (140.2, 111.8)
- added C14: 27nF, Capacitor_SMD:C_0805_2012Metric_Pad1.18x1.45mm_HandSolder, F.Cu at (111.8, 94.2)
- added C6: 10nF, Capacitor_SMD:C_0805_2012Metric, F.Cu at (114.1, 101.8)
- added C7: 100uF, Capacitor_SMD:CP_Elec_3x5.3, F.Cu at (140.2, 96.8)
- added C8: 1nF, Capacitor_SMD:C_0805_2012Metric, F.Cu at (114.1, 99.2)
- added C9: 47uF, Capacitor_SMD:C_0805_2012Metric_Pad1.18x1.45mm_HandSolder, F.Cu at (132.9, 104.8)
- added D32: BAT54SW, Package_TO_SOT_SMD:SOT-323_SC-70, F.Cu at (122.0, 113.7)
- added JP1: OSC_switch, Jumper:SolderJumper-2_P1.3mm_Open_RoundedPad1.0x1.5mm, F.Cu at (135.9, 97.8)
- added R3: 62k, Resistor_SMD:R_0805_2012Metric, F.Cu at (139.5, 84.8)
- added R4: 10k, Resistor_SMD:R_0805_2012Metric, F.Cu at (121.2, 110.5)
- added R5: 100k, Resistor_SMD:R_0805_2012Metric, F.Cu at (123.5, 110.5)
- added R8: 0.027, Resistor_SMD:R_0805_2012Metric, F.Cu at (115.8, 94.2)
- added TP1: TestPoint, TestPoint:TestPoint_Pad_D1.5mm, F.Cu at (110.5, 104.2)
- added TP2: TestPoint, TestPoint:TestPoint_Pad_D1.5mm, F.Cu at (118.0, 101.8)
- added TP3: ~, TestPoint:TestPoint_Pad_D1.5mm, F.Cu at (137.9, 91.2)
- added U3: LT4256-1CS8, LT4256-1CS8:SO-8_S, F.Cu at (112.8, 89.2)
- added U4: LM324, LM324DRG3:SOIC127P600X175-14N, F.Cu at (129.5, 113.5)
- C1: value 100uF -> 10nF; footprint Capacitor_SMD:CP_Elec_3x5.3 -> Capacitor_SMD:C_0805_2012Metric_Pad1.18x1.45mm_HandSolder
- C2: value 100nF -> 100uF; footprint Capacitor_SMD:C_0805_2012Metric -> Capacitor_SMD:CP_Elec_3x5.3
- C3: value 10nF -> 100uF; footprint Capacitor_SMD:C_0805_2012Metric -> Capacitor_SMD:CP_Elec_3x5.3
- C4: value 1nF -> 100nF
- C5: value 27nF -> 10nF
- J1: value Conn_01x02_Pin -> dcConn
- J2: value gateBias -> gateConn
- J3: value gateBias -> drainConn
- R2: value 0.027 -> 100k
- R6: value 100k -> 27k
- R7: value 27k -> 100k
- R9: value 30k -> 100k
- RV1: value 100k -> 200k
- U1: value LT4256-1CS8 -> LDO40LPURY; footprint LT4256-1CS8:SO-8_S -> LDO40LPURY:SON95P300X300X100-7N
- U2: value TPS7A1650DGNR -> LM2662MX_NOPB; footprint TPS7A1650DGNR:SOP65P490X110-9N -> LM2662MX_NOPB:SOIC127P599X175-8N
- moved R6 131.0 mm to (112.1, 84.2), turned to 180 degrees
- moved R9 130.9 mm to (122.0, 116.2), turned to 180 degrees
- moved J1 125.9 mm to (115.8, 115.8)
- moved R7 125.6 mm to (115.8, 84.2), turned to 180 degrees
- moved R1 124.8 mm to (114.1, 106.8), turned to 0 degrees
- moved D1 119.1 mm to (121.2, 86.0), turned to 0 degrees
- moved C2 117.9 mm to (114.1, 110.2), turned to 0 degrees
- moved RV1 117.0 mm to (135.5, 83.8)
- moved C4 113.6 mm to (114.1, 104.2), turned to 0 degrees
- moved Q1 111.7 mm to (121.5, 91.5), turned to -90 degrees
- moved J3 109.7 mm to (119.3, 81.7), turned to 0 degrees
- moved J2 108.0 mm to (138.4, 116.8)
- moved U2 106.9 mm to (138.2, 104.2), turned to 0 degrees
- moved C1 103.8 mm to (134.0, 91.2), turned to 0 degrees
- moved C3 102.8 mm to (130.0, 88.8), turned to 180 degrees
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Connections:
- C5 pad 1: Net-(U1-TIMER) -> posGateV
- J1 pad 2: drainV -> +28V
- J3 pad 2: +28V -> drainV
- Q1 pad 5_8: Net-(U1-SENSE) -> Net-(U3-SENSE)
- R2 pad 1: +28V -> posGateV
- R2 pad 2: Net-(U1-SENSE) -> Net-(U1-ADJ)
- R6 pad 1: drainV -> Net-(U3-FB)
- R6 pad 2: Net-(U1-FB) -> GND
- R7 pad 1: Net-(U1-FB) -> drainV
- R7 pad 2: GND -> Net-(U3-FB)
- R9 pad 1: Net-(U2-FB/DNC) -> isGateOn
- R9 pad 2: Net-(R9-Pad2) -> Net-(D32-A)
- RV1 pad 1: Net-(R9-Pad2) -> Net-(R3-Pad2)
- U1 pad 1: isGateOn -> GND
- U1 pad 2: Net-(U1-FB) -> +28V
- U1 pad 3: Net-(U1-PWRGD) -> +28V
- U1 pad 4: GND -> posGateV
- U1 pad 5: Net-(U1-TIMER) -> posGateV
- U1 pad 6: Net-(D1-K) -> Net-(U1-ADJ)
- U1 pad 7: Net-(U1-SENSE) -> (no net)
- U2 pad 1: posGateV -> Net-(JP1-B)
- U2 pad 2: Net-(U2-FB/DNC) -> Net-(U2-CAP+)
- U2 pad 3: Net-(U2-PG) -> GND
- U2 pad 4: GND -> Net-(U2-CAP-)
- U2 pad 5: +28V -> negGateV
- U2 pad 6: (no net) -> GND
- U2 pad 7: Net-(U2-DELAY) -> unconnected-(U2-OSC-Pad7)
- U2 pad 8: +28V -> posGateV
Routing:
- net +28V: track 56.3 -> 16.7 mm
- net Net-(U1-SENSE): track 23.1 -> 0.00 mm, vias 2 -> 0
- net Net-(U1-FB): track 21.9 -> 0.00 mm, vias 2 -> 0
- net isGateOn: track 1.82 -> 22.6 mm
- net Net-(U3-SENSE): track 0.00 -> 16.8 mm
- net Net-(U2-FB/DNC): track 12.7 -> 0.00 mm, vias 2 -> 0
- net Net-(D32-A): track 0.00 -> 11.7 mm
- net Net-(U2-PG): track 10.5 -> 0.00 mm
- net Net-(U32-CAP+): track 8.11 -> 0.00 mm
- net Net-(JP1-B): track 0.00 -> 8.08 mm
- net Net-(JP32-B): track 8.01 -> 0.00 mm
- net Net-(U32-CAP-): track 7.78 -> 0.00 mm
- net Net-(U1-ADJ): track 0.00 -> 6.72 mm
- net posGateV: track 38.8 -> 32.2 mm
- net Net-(U4A--): track 0.00 -> 5.96 mm
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- removed copper zone on B.Cu, net GND

Commit message: init idea
Parts:
- removed C3: 100uF, Capacitor_SMD:CP_Elec_3x5.3
- added TP4: TestPoint, TestPoint:TestPoint_Pad_D1.5mm, F.Cu at (134.0, 71.0)
- added TP5: TestPoint, TestPoint:TestPoint_Pad_D1.5mm, F.Cu at (125.4, 62.3)
- U1: footprint LDO40LPURY:SON95P300X300X100-7N -> Package_DFN_QFN:DFN-6-1EP_3x3mm_P0.95mm_EP1.7x2.6mm
- moved J2 61.8 mm to (136.0, 55.0)
- moved U4 56.0 mm to (146.5, 60.1), turned to 90 degrees
- moved R9 55.7 mm to (149.3, 67.6), turned to -90 degrees
- moved D32 52.3 mm to (146.8, 67.6), turned to 90 degrees
- moved R5 48.6 mm to (143.5, 66.2), turned to 0 degrees
- moved R4 47.6 mm to (143.5, 68.4), turned to 180 degrees
- moved C12 37.3 mm to (150.0, 72.8)
- moved C13 37.3 mm to (150.0, 75.8)
- moved C2 32.1 mm to (130.4, 82.5)
- moved C4 32.1 mm to (130.4, 76.5)
- moved C6 32.1 mm to (130.4, 74.0)
- moved C8 32.1 mm to (130.4, 71.5)
- moved J1 32.1 mm to (132.1, 88.0)
- moved R1 32.1 mm to (130.4, 79.0)
- moved TP1 32.1 mm to (126.8, 76.5)
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Connections:
- U1 pad 7: (no net) -> GND
Routing:
- net +28V: track 16.7 -> 71.7 mm, vias 0 -> 2
- net isGateOn: track 22.6 -> 61.7 mm, vias 0 -> 2
- net negGateV: track 13.6 -> 51.1 mm
- net posGateV: track 32.2 -> 53.5 mm, vias 0 -> 2
- net Net-(R3-Pad2): track 4.04 -> 15.0 mm
- net Net-(U3-PWRGD): track 0.00 -> 5.46 mm
- net Net-(JP1-B): track 8.08 -> 4.83 mm
- net drainV: track 19.9 -> 20.5 mm
- net GND: vias 0 -> 261
- added copper zone on B.Cu, net GND
Other:
- board outline added: 33.2 x 41.3 mm

Commit message: init idea
Routing:
- net posGateV: track 53.5 -> 52.9 mm
Changed lines of the file:
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@@
 		(tenting front back)
 		(pcbplotparams
-			(layerselection 0x00000000_00000000_55555555_5755f5ff)
+			(layerselection 0x00000000_00000000_55555555_575555ff)
 			(plot_on_all_layers_selection 0x00000000_00000000_00000000_00000000)
 			(disableapertmacros no)
@@
 			(usegerberadvancedattributes yes)
 			(creategerberjobfile yes)
+			(gerberprecision 5)
 			(dashed_line_dash_ratio 12.000000)
 			(dashed_line_gap_ratio 3.000000)
@@
 			(plotframeref no)
 			(mode 1)
-			(useauxorigin no)
+			(useauxorigin yes)
 			(hpglpennumber 1)
 			(hpglpenspeed 20)
@@
 			(outputformat 1)
 			(mirror no)
-			(drillshape 1)
+			(drillshape 0)
 			(scaleselection 1)
-			(outputdirectory "")
+			(outputdirectory "mfg/")
 		)
 	)
@@
 		(at 129.0875 63.2 -90)
 		(property "Reference" "U3"
-			(at -2.9 -4.3 270)
+			(at -0.1 -3.6125 270)
 			(unlocked yes)
 			(layer "F.SilkS")
@@
 		)
 		(fill no)
+		(locked yes)
 		(layer "Edge.Cuts")
 	)
@@
 	)
 	(segment
-		(start 140.9875 75.25)
-		(end 142.2075 74.03)
-		(width 0.2)
-		(layer "F.Cu")
-		(net 2)
-	)
-	(segment
 		(start 140.6375 73.15)
 		(end 140.8375 72.95)
@@
 	)
 	(segment
+		(start 142.2075 74.03)
+		(end 142.2075 72.93)
+		(width 0.2)
+		(layer "F.Cu")
+		(net 2)
+	)
+	(segment
 		(start 146.95 86.95)
 		(end 147.15 87.15)
@@
 	)
 	(segment
+		(start 140.9875 75.25)
+		(end 142.2075 74.03)
+		(width 0.2)
+		(layer "F.Cu")
+		(net 2)
+	)
+	(segment
+		(start 139.6375 77.05)
+		(end 140.9375 77.05)
+		(width 0.2)
+		(layer "F.Cu")
+		(net 2)
+	)
+	(segment
 		(start 149.1 87.9)
 		(end 149.1375 87.8625)
@@
 	)
 	(segment
-		(start 142.2075 74.03)
-		(end 142.2075 72.93)
+		(start 148.2875 89.2)
+		(end 148.65 88.8375)
 		(width 0.2)
 		(layer "F.Cu")
@@
 	)
 	(segment
-		(start 148.2875 89.2)
-		(end 148.65 88.8375)
+		(start 140.9875 77)
+		(end 140.9875 75.25)
 		(width 0.2)
 		(layer "F.Cu")
@@
 	)
 	(segment
-		(start 139.6375 76.45)
-		(end 139.6375 77.05)
-		(width 0.2)
-		(layer "F.Cu")
-		(net 2)
-	)
-	(segment
 		(start 141.1375 71.35)
 		(end 142.0625 71.35)
@@
 	)
 	(segment
-		(start 139.7375 76.35)
-		(end 139.6375 76.45)
-		(width 0.2)
-		(layer "F.Cu")
-		(net 2)
-	)
-	(segment
-		(start 140.9875 76.35)
-		(end 140.9875 75.25)
+		(start 137.4875 73.7)
+		(end 138.0375 73.15)
 		(width 0.2)
 		(layer "F.Cu")
@@
 	)
 	(segment
-		(start 137.4875 73.7)
-		(end 138.0375 73.15)
+		(start 140.9375 77.05)
+		(end 140.9875 77)
 		(width 0.2)
 		(layer "F.Cu")
@@
 	)
 	(segment
-		(start 140.9875 76.35)
-		(end 139.7375 76.35)
-		(width 0.2)
-		(layer "F.Cu")
-		(net 2)
-	)
-	(segment
 		(start 152.8375 82.95)
 		(end 151.3375 82.95)
@@
 	)
 	(via
-		(at 140.9875 76.35)
+		(at 140.9875 77)
 		(size 0.6)
 		(drill 0.3)
@@
 	)
 	(segment
-		(start 140.1875 82.75)
-		(end 140.1875 89.05)
+		(start 140.9875 77)
+		(end 140.9875 81.95)
 		(width 0.2)
 		(layer "B.Cu")
@@
 	)
 	(segment
-		(start 140.3375 89.2)
-		(end 146.1375 89.2)
+		(start 140.1875 89.05)
+		(end 140.3375 89.2)
 		(width 0.2)
 		(layer "B.Cu")
@@
 	)
 	(segment
-		(start 140.9875 76.35)
-		(end 140.9875 81.95)
+		(start 140.3375 89.2)
+		(end 146.1375 89.2)
 		(width 0.2)
 		(layer "B.Cu")
@@
 	)
 	(segment
-		(start 140.1875 89.05)
-		(end 140.3375 89.2)
+		(start 140.1875 82.75)
+		(end 140.1875 89.05)
 		(width 0.2)
 		(layer "B.Cu")
@@
 		(net 1)
 		(net_name "GND")
+		(locked yes)
 		(layers "F.Cu" "B.Cu")
 		(name "gnd_plane")

Commit message: init ideas
Parts:
- moved TP2 108.5 mm to (219.4, 128.0)
- moved C1 108.5 mm to (234.1, 143.3)
- moved C10 108.5 mm to (237.5, 139.6)
- moved C11 108.5 mm to (241.4, 143.3)
- moved C14 108.5 mm to (220.8, 124.6)
- moved C2 108.5 mm to (223.2, 138.9)
- moved C4 108.5 mm to (223.2, 132.9)
- moved C5 108.5 mm to (232.1, 130.6)
- moved C6 108.5 mm to (223.2, 130.4)
- moved C7 108.5 mm to (229.1, 131.6)
- moved C8 108.5 mm to (223.2, 128.0)
- moved C9 108.5 mm to (237.5, 137.1)
- moved D1 108.5 mm to (230.3, 116.3)
- moved D32 108.5 mm to (239.5, 124.0)
- moved J1 108.5 mm to (224.8, 144.4)
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