File: GaN_pwr_delivery_module.kicad_pcb (KiCad board)
At the start: 2 copper layers, 33.2 x 41.3 mm, 39 parts, among them J1 dcConn, J2 gateConn, J3 drainConn, Q1 AONS66920, U1 LDO40LPURY, U2 LM2662MX_NOPB, U3 LT4256-1CS8, U4 LM324

Commit message: POC
Parts:
- removed C13, C7: 100uF, Capacitor_SMD:CP_Elec_3x5.3
- added TP6: TestPoint, TestPoint:TestPoint_Pad_D1.5mm, F.Cu at (242.7, 132.5)
- C2: footprint Capacitor_SMD:CP_Elec_3x5.3 -> Capacitor_SMD:CP_Elec_6.3x9.9
- TP3: value ~ -> TestPoint
- moved C2 1.56 mm to (222.4, 140.3)
- moved J1 0.75 mm to (224.9, 145.2)
Connections:
- U4 pad 6: unconnected-(U4B---Pad6) -> unconnected-(U4B-+-Pad5)
Routing:
- net +28V: track 71.7 -> 75.7 mm, vias 2 -> 3
- net posGateV: track 52.9 -> 49.6 mm
- net negGateV: track 51.1 -> 51.7 mm
- net GND: vias 261 -> 276
Other:
- board text added: "C"
- board text added: "v1.1"
