File: GaN_pwr_delivery_module.kicad_pcb (KiCad board)
At the start: 2 copper layers, 33.2 x 41.3 mm, 38 parts, among them J1 dcConn, J2 gateConn, J3 drainConn, Q1 AONS66920, U1 LDO40LPURY, U2 LM2662MX_NOPB, U3 LT4256-1CS8, U4 LM324

Commit message: POC
Parts:
- added C32: 10uF, Capacitor_SMD:CP_Elec_6.3x9.9, F.Cu at (194.6, 92.9)
- added C33: 22uF, Capacitor_SMD:CP_Elec_6.3x9.9, F.Cu at (198.5, 107.4)
- added C34: 10nF, Capacitor_SMD:C_0805_2012Metric_Pad1.18x1.45mm_HandSolder, F.Cu at (173.7, 108.2)
- added D33: BAT54SW, Package_TO_SOT_SMD:SOT-323_SC-70, F.Cu at (177.4, 112.7)
- added D34: BAT54SW, Package_TO_SOT_SMD:SOT-323_SC-70, F.Cu at (185.4, 95.3)
- added R32: 100k, Resistor_SMD:R_0805_2012Metric, F.Cu at (188.4, 95.3)
- added R33: 62k, Resistor_SMD:R_0805_2012Metric, F.Cu at (185.5, 91.9)
- added RV32: 200k, Potentiometer_THT:Potentiometer_Bourns_3296W_Vertical, F.Cu at (180.4, 93.6)
- added U32: LM317D2T, LM317D2T:VREG_L7805ACD2T, F.Cu at (185.2, 104.5)
Routing:
- net Net-(D33-A): track 0.00 -> 39.9 mm
- net Net-(D34-A): track 0.00 -> 33.3 mm
- net Net-(D33-K): track 0.00 -> 13.3 mm
- net Net-(R33-Pad2): track 0.00 -> 4.88 mm
Other:
- board outline removed
